File: ESP32S3_M.2_Board/ESP32S3_M.2_Board.kicad_pcb (KiCad board)
At the start: 4 copper layers, 23 x 42 mm, 55 parts, among them J1 USB_C_Receptacle_USB2.0, J2 M.2-B-KEY, U1 TLV62568DBV, U2 USBLC6-2SC6, U3 ESP32-S3R8, U4 W25Q16JVUXIQ, Y1 40MHz, Y2 32.768KHz

Commit message: Firmware Adding
Other:
- board text removed: "PCB32_BR_ESP32S3_M.2_Board"
- board text removed: "PCB32_TL_ESP32S3_M.2_Board"
Changed lines of the file:
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@@
 			)
 		)
-		(property "Footprint" ""
+		(property "Footprint" "LOGO"
 			(at 0 0 0)
 			(unlocked yes)
@@
 		)
 	)
-	(gr_text "PCB32_TL_ESP32S3_M.2_Board"
-		(at 213.625 87.125 0)
-		(layer "F.SilkS")
-		(effects
-			(font
-				(size 1.5 1.5)
-				(thickness 0.3)
-				(bold yes)
-			)
-			(justify left bottom)
-		)
-	)
 	(gr_text "M.2 USB\nENABLE\n"
 		(at 232.625 123.4 0)
@@
 				(bold yes)
 			)
-			(justify left bottom)
-		)
-	)
-	(gr_text "PCB32_BR_ESP32S3_M.2_Board"
-		(at 243 136.05 0)
-		(layer "F.SilkS")
-		(effects
-			(font
-				(size 1.5 1.5)
-				(thickness 0.3)
-				(bold yes)
-			)

Commit message: feat: push for v.2
Parts:
- removed the R10 at (237.9, 128.8)
- removed R13: 10k, Resistor_SMD:R_0201_0603Metric_Pad0.64x0.40mm_HandSolder
- removed the R3 at (239.6, 107.2)
- added D1: LED, LED_SMD:LED_0402_1005Metric_Pad0.77x0.64mm_HandSolder, B.Cu at (236.6, 107.2)
- added D2: LED, LED_SMD:LED_0402_1005Metric_Pad0.77x0.64mm_HandSolder, B.Cu at (236.6, 108.3)
- added JP1: 3V3_M2, Resistor_SMD:R_0201_0603Metric, F.Cu at (237.9, 128.4)
- added JP2: VBUS_M2, Resistor_SMD:R_0201_0603Metric, B.Cu at (237.7, 128.1)
- added R5: 22R, Resistor_SMD:R_0402_1005Metric_Pad0.72x0.64mm_HandSolder, F.Cu at (239.6, 106.6)
- added R8: 100k, Resistor_SMD:R_0402_1005Metric_Pad0.72x0.64mm_HandSolder, B.Cu at (236.8, 117.3)
- added TP1: TestPoint, TestPoint:TestPoint_Pad_D1.0mm, B.Cu at (229.7, 117.7)
- added TP10: TestPoint, TestPoint:TestPoint_Pad_D1.0mm, F.Cu at (227.5, 103.2)
- added TP2: TestPoint, TestPoint:TestPoint_Pad_D1.0mm, B.Cu at (231.4, 116.4)
- added TP3: TestPoint, TestPoint:TestPoint_Pad_D1.0mm, B.Cu at (238.6, 118.2)
- added TP4: TestPoint, TestPoint:TestPoint_Pad_D1.0mm, B.Cu at (237.2, 121.8)
- added TP5: TestPoint, TestPoint:TestPoint_Pad_D1.0mm, F.Cu at (219.2, 112.2)
- added TP7: TestPoint, TestPoint:TestPoint_Pad_D1.0mm, F.Cu at (230.8, 103.8)
- added TP8: TestPoint, TestPoint:TestPoint_Pad_D1.0mm, B.Cu at (238.1, 113.9)
- added TP9: TestPoint, TestPoint:TestPoint_Pad_D1.0mm, F.Cu at (235.3, 117.3)
- ANT1: value 2450AT18B100E -> KH-3216-H0209; footprint SamacSys_Parts:ANTC3216X140N -> PCB_Lib_DaanHeetkamp_KiCad:ANTC3216X140N
- J1: value USB_C_Receptacle_USB2.0 -> USB-C
- LED1: renamed from LED; value WS2812C-2020 -> WS2812C-2020-V1
- R12: moved to B.Cu
- U2: renamed from U1; value TLV62568DBV -> TLV62568DBVR
- moved R11 21.3 mm to (238.4, 106.7), turned to -90 degrees
- moved G*** 15.3 mm to (222.5, 121.0)
- moved R12 5.69 mm to (238.4, 109.0), turned to 90 degrees
- moved R4 3.56 mm to (232.4, 119.3), turned to -45 degrees
- moved R3 2.89 mm to (231.8, 119.9), turned to -45 degrees
- moved C20 1.01 mm to (235.3, 117.3)
- moved C17 0.92 mm to (234.2, 117.3)
- moved R6 0.45 mm to (234.9, 93.2)
- moved R7 0.40 mm to (234.9, 94.5)
- moved R1 0.23 mm to (222.7, 94.2)
- moved R2 0.22 mm to (220.2, 94.2)
- moved U1 0.22 mm to (229.1, 103.2), turned to -90 degrees
- renumbered BOOT to BOOT1, C16 to C1, C3 to C10, C24 to C12, C12 to C13, C13 to C14, C25 to C15, C14 to C16, C21 to C17, C15 to C18, C6 to C19, C17 to C2, C22 to C20, C7 to C21, C8 to C22, C26 to C23, C9 to C24, C10 to C25, C23 to C26, C18 to C3, C19 to C4, C20 to C5, C4 to C6, C5 to C7, C1 to C8, C2 to C9, L2 to L1, L1 to L2, R7 to R1, R9 to R10, R8 to R2, R1 to R3, R2 to R4, R4 to R6, R6 to R7, R5 to R9, RST to RST1, U2 to U1
Connections:
- R11 pad 1: Net-(J2-2) -> VBUS
- R11 pad 2: VBUS -> Net-(D1-A)
- R12 pad 2: /CHIP_BOOT -> Net-(D2-A)
- U1 pad 1: /USB_D+ -> /USB_D-
- U1 pad 4: /USB_D- -> /USB_D+
Routing:
- net Earth: track 124.6 -> 144.0 mm, vias 49 -> 45
- net /USB_D-: track 37.9 -> 30.7 mm
- net +3V3: track 25.1 -> 30.3 mm
- net /USB_D+: track 40.6 -> 36.0 mm
- net VDD_SPI: track 10.1 -> 14.6 mm, vias 2 -> 3
- net /GPIO46: track 39.7 -> 44.0 mm
- net /FLASH_QSPI_nCS: track 6.04 -> 9.52 mm, vias 0 -> 1
- net /M.2_USB_D+: track 9.56 -> 13.0 mm
- net /M.2_USB_D-: track 9.40 -> 12.6 mm
- net +3V3_RF: track 12.7 -> 14.4 mm
- net Net-(D2-A): track 0.00 -> 1.30 mm
- net Net-(D1-A): track 0.00 -> 1.28 mm
- net /GPIO45: track 31.4 -> 30.2 mm
- net VBUS: track 50.4 -> 49.1 mm
- net Net-(U2-EN): track 13.9 -> 13.0 mm
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Other:
- board text added: "BOOT"
- board text added: "ESP32S3.M.2 D.Heetkamp 27-2-25 V2"
- board text added: "RGB IO46"
- board text added: "RST"
- board text removed: "ESP32S3.M.2 D.Heetkamp 17-4-24"
- board text removed: "STRAP"
