File: ESP32S3_M.2_Board/ESP32S3_M.2_Board.kicad_sch (KiCad schematic)
At the start: 54 parts, among them J1 USB_C_Receptacle_USB2.0, J2 M.2-B-KEY, U1 TLV62568DBV, U2 USBLC6-2SC6, U3 ESP32-S3R8, U4 W25Q16JVUXIQ, Y1 40MHz, Y2 32.768KHz

Commit message: feat: push for v.2
Parts:
- removed R10: 10k, Resistor_SMD:R_0402_1005Metric_Pad0.72x0.64mm_HandSolder, symbol Device:R
- removed R13, R3: 10k, Resistor_SMD:R_0201_0603Metric_Pad0.64x0.40mm_HandSolder, symbol Device:R
- added D1, D2: LED, LED_SMD:LED_0402_1005Metric_Pad0.77x0.64mm_HandSolder, symbol Device:LED
- added JP1: 3V3_M2, Resistor_SMD:R_0201_0603Metric, symbol Jumper:SolderJumper_2_Open
- added JP2: VBUS_M2, Resistor_SMD:R_0201_0603Metric, symbol Jumper:SolderJumper_2_Open
- added R5: 22R, Resistor_SMD:R_0402_1005Metric_Pad0.72x0.64mm_HandSolder, symbol Device:R
- added R8: 100k, Resistor_SMD:R_0402_1005Metric_Pad0.72x0.64mm_HandSolder, symbol Device:R
- added TP1, TP10, TP2, TP3, TP4, TP5, TP7, TP8, TP9: TestPoint, TestPoint:TestPoint_Pad_D1.0mm, symbol Connector:TestPoint
- ANT1: value 2450AT18B100E -> KH-3216-H0209; footprint SamacSys_Parts:ANTC3216X140N -> PCB_Lib_DaanHeetkamp_KiCad:ANTC3216X140N; LCSC PART # (none) -> C2925417; Manufacturer_Name JOHANSON TECHNOLOGY -> Shenzhen Kinghelm Elec; Manufacturer_Part_Number 2450AT18B100E -> KH-3216-H0209
- BOOT1, RST1: LCSC PART # (none) -> C512395; Manufacturer_Name (none) -> PANASONIC; Manufacturer_Part_Number (none) -> EVQP2P02W
- C1: renamed from C16; LCSC PART # (none) -> C82453; Manufacturer_Name (none) -> Murata Electronics; Manufacturer_Part_Number (none) -> GRM155R60J475ME47D
- C10: renamed from C3; LCSC PART # (none) -> C2992625; Manufacturer_Name (none) -> FH (Guangdong Fenghua Advanced Tech); Manufacturer_Part_Number (none) -> 0402X106M100CT
- C11: LCSC PART # (none) -> C113791; Manufacturer_Name (none) -> KDS Daishinku; Manufacturer_Part_Number (none) -> CC0402MRX5R6BB105
- C12: renamed from C24; LCSC PART # (none) -> C1660; Manufacturer_Name (none) -> Darfon Elec; Manufacturer_Part_Number (none) -> 0603CG3R3C500NT
- C13: renamed from C12; LCSC PART # (none) -> C361203; Manufacturer_Name (none) -> YAGEO; Manufacturer_Part_Number (none) -> C1005X5R1E104KT000E
- C14: renamed from C13; LCSC PART # (none) -> C361203; Manufacturer_Name (none) -> YAGEO; Manufacturer_Part_Number (none) -> C1005X5R1E104KT000E
- C15: renamed from C25; LCSC PART # (none) -> C1660; Manufacturer_Name (none) -> Darfon Elec; Manufacturer_Part_Number (none) -> 0603CG3R3C500NT
- C16: renamed from C14; LCSC PART # (none) -> C361203; Manufacturer_Name (none) -> YAGEO; Manufacturer_Part_Number (none) -> C1005X5R1E104KT000E
- C17: renamed from C21; LCSC PART # (none) -> C361203; Manufacturer_Name (none) -> YAGEO; Manufacturer_Part_Number (none) -> C1005X5R1E104KT000E
- C18: renamed from C15; LCSC PART # (none) -> C361203; Manufacturer_Name (none) -> YAGEO; Manufacturer_Part_Number (none) -> C1005X5R1E104KT000E
- C19: renamed from C6; LCSC PART # (none) -> C258501; Manufacturer_Name (none) -> TDK; Manufacturer_Part_Number (none) -> C1005NP0100JGTS
- C2: renamed from C17; LCSC PART # (none) -> C361203; Manufacturer_Name (none) -> YAGEO; Manufacturer_Part_Number (none) -> C1005X5R1E104KT000E
- C20: renamed from C22; LCSC PART # (none) -> C113791; Manufacturer_Name (none) -> KDS Daishinku; Manufacturer_Part_Number (none) -> CC0402MRX5R6BB105
- C21: renamed from C7; LCSC PART # (none) -> C258501; Manufacturer_Name (none) -> TDK; Manufacturer_Part_Number (none) -> C1005NP0100JGTS
- C22: renamed from C8; LCSC PART # (none) -> C107000; Manufacturer_Name (none) -> YAGEO; Manufacturer_Part_Number (none) -> CC0402JRNPO9BN200
- C23: renamed from C26; LCSC PART # (none) -> C361203; Manufacturer_Name (none) -> YAGEO; Manufacturer_Part_Number (none) -> C1005X5R1E104KT000E
- C24: renamed from C9; LCSC PART # (none) -> C107000; Manufacturer_Name (none) -> YAGEO; Manufacturer_Part_Number (none) -> CC0402JRNPO9BN200
- C25: renamed from C10; LCSC PART # (none) -> C361203; Manufacturer_Name (none) -> YAGEO; Manufacturer_Part_Number (none) -> C1005X5R1E104KT000E
- C26: renamed from C23; LCSC PART # (none) -> C361203; Manufacturer_Name (none) -> YAGEO; Manufacturer_Part_Number (none) -> C1005X5R1E104KT000E
- C3: renamed from C18; LCSC PART # (none) -> C361203; Manufacturer_Name (none) -> YAGEO; Manufacturer_Part_Number (none) -> C1005X5R1E104KT000E
- C4: renamed from C19; LCSC PART # (none) -> C361203; Manufacturer_Name (none) -> YAGEO; Manufacturer_Part_Number (none) -> C1005X5R1E104KT000E
- C5: renamed from C20; LCSC PART # (none) -> C82453; Manufacturer_Name (none) -> Murata Electronics; Manufacturer_Part_Number (none) -> GRM155R60J475ME47D
- C6: renamed from C4; LCSC PART # (none) -> C82453; Manufacturer_Name (none) -> Murata Electronics; Manufacturer_Part_Number (none) -> GRM155R60J475ME47D
- C7: renamed from C5; LCSC PART # (none) -> C2992625; Manufacturer_Name (none) -> FH (Guangdong Fenghua Advanced Tech); Manufacturer_Part_Number (none) -> 0402X106M100CT
- C8: renamed from C1; LCSC PART # (none) -> C361203; Manufacturer_Name (none) -> YAGEO; Manufacturer_Part_Number (none) -> C1005X5R1E104KT000E
- C9: renamed from C2; LCSC PART # (none) -> C361203; Manufacturer_Name (none) -> YAGEO; Manufacturer_Part_Number (none) -> C1005X5R1E104KT000E
- J1: value USB_C_Receptacle_USB2.0 -> USB-C; LCSC PART # (none) -> C136423; Manufacturer_Name (none) -> SOFNG; Manufacturer_Part_Number (none) -> MC-311D
- L1: renamed from L2; LCSC PART # (none) -> C135262; Manufacturer_Name (none) -> SXN(Shun Xiang Nuo Elec); Manufacturer_Part_Number (none) -> SMNR4020-2.2UH
- L2: renamed from L1; LCSC PART # (none) -> C29682; Manufacturer_Name (none) -> Sunlord; Manufacturer_Part_Number (none) -> SDCL1608C2N2STDF
- L3: LCSC PART # (none) -> C29682; Manufacturer_Name (none) -> Sunlord; Manufacturer_Part_Number (none) -> SDCL1608C2N2STDF
- LED1: value WS2812C-2020 -> WS2812C-2020-V1; LCSC PART # (none) -> C2976072
- R1: renamed from R7; LCSC PART # (none) -> C105873; Manufacturer_Name (none) -> YAGEO; Manufacturer_Part_Number (none) -> RC0402JR-075K1L
- R10: renamed from R9; LCSC PART # (none) -> C163810; Manufacturer_Name (none) -> Walsin Tech Corp; Manufacturer_Part_Number (none) -> WR04X1002FTL
- R11: LCSC PART # (none) -> C163810; Manufacturer_Name (none) -> Walsin Tech Corp; Manufacturer_Part_Number (none) -> WR04X1002FTL; now fitted; now in the parts list
- R12: LCSC PART # (none) -> C163810; Manufacturer_Name (none) -> Walsin Tech Corp; Manufacturer_Part_Number (none) -> WR04X1002FTL
- R2: renamed from R8; LCSC PART # (none) -> C105873; Manufacturer_Name (none) -> YAGEO; Manufacturer_Part_Number (none) -> RC0402JR-075K1L
- R6: renamed from R4; LCSC PART # (none) -> C5159688; Manufacturer_Name (none) -> FOJAN; Manufacturer_Part_Number (none) -> FRC0402F4503TS
- R7: renamed from R6; LCSC PART # (none) -> C705662; Manufacturer_Name (none) -> YAGEO; Manufacturer_Part_Number (none) -> RT0402CRE07100KL
- R9: renamed from R5; LCSC PART # (none) -> C413049; Manufacturer_Name (none) -> Espressif Systems; Manufacturer_Part_Number (none) -> ERJ2RKF22R0X
- U1: renamed from U2; LCSC PART # (none) -> C2827654; Manufacturer_Name (none) -> TECH PUBLIC; Manufacturer_Part_Number (none) -> USBLC6-2SC6
- U2: renamed from U1; value TLV62568DBV -> TLV62568DBVR; LCSC PART # (none) -> C163219; Manufacturer_Name (none) -> Texas Instruments; Manufacturer_Part_Number (none) -> TLV62568DBVR
- U3: LCSC PART # (none) -> C2913194; Manufacturer_Name (none) -> Espressif Systems; Manufacturer_Part_Number (none) -> ESP32-S3R8
- U4: LCSC PART # (none) -> C2843335; Manufacturer_Name (none) -> Winbond Elec; Manufacturer_Part_Number (none) -> W25Q16JVUXIQ
- Y1: LCSC PART # (none) -> C2885592; Manufacturer_Name (none) -> YXC Crystal Oscillators; Manufacturer_Part_Number (none) -> X252040MMB4SI
- Y2: LCSC PART # (none) -> C93232; Manufacturer_Name (none) -> PANASONIC; Manufacturer_Part_Number (none) -> DST310S 32.768KHz
- renumbered R1 to R3, R2 to R4
Connections:
- net +3V3: now also JP1.2 (B), TP4.1, TP7.1
- net +3V3_RF: now also TP5.1
- net CHIP_BOOT: no longer R12.2
- net Earth: now also D1.1 (K), D2.1 (K)
- net FLASH_QSPI_nCS: now also R8.1, TP8.1
- net GPIO46: now also TP10.1
- net USB_D+: now also U1.4 (I/O2), TP2.1; no longer U1.1 (I/O1)
- net USB_D-: now also U1.1 (I/O1), TP1.1; no longer U1.4 (I/O2)
- net VBUS: now also R11.1, JP2.1 (A), R5.1, TP3.1; no longer R11.2
- net VDD_SPI: now also R8.2, TP9.1
- net at U2.1 (EN): now also R5.2
- net at J2.P$2 (2), J2.P$4 (4): now also JP2.2 (B); no longer R11.1
- net at J2.P$1 (1), J2.P$3 (3): now also JP1.1 (A)
- new net: D2.2 (A), R12.2
- new net: D1.2 (A), R11.2
Other:
- note added: "3V3_EXT"
- note added: "Boot Button"
- note added: "C113791"
- note added: "C56392"
- note added: "GPIO 1 and 46 HIGH = SPI Download Boot Mode - GPIO 45 = VDD_SPI Voltage LOW = VDD3P3_RTC HIGH = 1.8V internal LDO"
- note added: "NP = Normal P = Directly in Flash"
- note added: "Note: For the M.2 USB resistors 470 Ohm are removed."
- note added: "PWR_EN"
- note added: "Status LEDs"
- note added: "VBUS + 3V3"
- note added: "VBUS_EXT"
- note added: "https://github.com/lllucius/esp32_extflash"
- note removed: "BOOT Button"
- company: (none) -> LiberBoard
- title: (none) -> ESP32S3 M.2 SOM
- moved on the sheet: BOOT1, C26, C8, R3, R4, U1
